File: Starter.sch (EAGLE design)
At the start: 8 parts, among them IC1 LM317MBSTT3

Commit message: Nets connected
Connections:
- new net +5V: C1.1, C2.+, D1.A, D1.C, D2.C, IC1.IN, IC1.OUT, R1.2
- new net GND: C1.2, C2.-, C3.-, R2.1
- new net N$1: C3.+, D2.A, IC1.ADJ, R1.1, R2.2
Other:
- note added: "5V Voltage Regulator"
- note added: "C2 helps to improve transient response"
- note added: "C3 is for ripple rejection"
- note added: "D1 protects against input short circuit"
- note added: "D2 protects against input short circuit"
- note added: "Notes:"
- note added: "Vref = 1.25V"
- moved on the sheet: C1, C2, C3, D1, D2, IC1, R1, R2

Commit message: Connector added
Parts:
- added J1: (no value), con-amp:520250-1
Connections:
- net +5V: now also J1.1
- net GND: now also J1.2
Changed lines of the file:
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@@
 <part name="P+2" library="supply1" library_urn="urn:adsk.eagle:library:371" deviceset="+5V" device=""/>
 <part name="P+1" library="supply1" library_urn="urn:adsk.eagle:library:371" deviceset="+5V" device=""/>
+<part name="J1" library="con-amp" library_urn="urn:adsk.eagle:library:127" deviceset="520250-1" device="" package3d_urn="urn:adsk.eagle:package:8081424/1"/>
+<part name="P+3" library="supply1" library_urn="urn:adsk.eagle:library:371" deviceset="+5V" device=""/>
+<part name="GND1" library="supply1" library_urn="urn:adsk.eagle:library:371" deviceset="GND" device=""/>
 </parts>
 <sheets>
@@
 <text x="172.72" y="25.4" size="5.08" layer="94">Starter Project</text>
 <text x="185.42" y="7.62" size="5.08" layer="94">Revision 1</text>
-<text x="101.6" y="144.78" size="1.778" layer="97" align="center">5V Voltage Regulator</text>
+<text x="96.52" y="147.32" size="1.778" layer="97" align="center">5V Voltage Regulator</text>
 <wire x1="91.44" y1="124.46" x2="91.44" y2="115.57" width="0.1524" layer="97"/>
 <wire x1="91.44" y1="111.76" x2="91.44" y2="104.14" width="0.1524" layer="97"/>
@@
 <attribute name="VALUE" x="109.22" y="137.16" size="1.778" layer="96" rot="R180"/>
 </instance>
+<instance part="J1" gate="G$1" x="121.92" y="137.16" smashed="yes">
+<attribute name="NAME" x="121.92" y="142.24" size="1.778" layer="95"/>
+<attribute name="VALUE" x="119.38" y="134.112" size="1.778" layer="96"/>
+</instance>
+<instance part="P+3" gate="1" x="116.84" y="147.32" smashed="yes">
+<attribute name="VALUE" x="114.3" y="142.24" size="1.778" layer="96" rot="R90"/>
+</instance>
+<instance part="GND1" gate="1" x="116.84" y="132.08" smashed="yes">
+<attribute name="VALUE" x="114.3" y="129.54" size="1.778" layer="96"/>
+</instance>
 </instances>
 <busses>
@@
 <wire x1="106.68" y1="106.68" x2="106.68" y2="99.06" width="0.1524" layer="91"/>
 <pinref part="SUPPLY4" gate="1" pin="GND"/>
+</segment>
+<segment>
+<pinref part="GND1" gate="1" pin="GND"/>
+<wire x1="116.84" y1="134.62" x2="116.84" y2="137.16" width="0.1524" layer="91"/>
+<pinref part="J1" gate="G$1" pin="2"/>
+<wire x1="116.84" y1="137.16" x2="119.38" y2="137.16" width="0.1524" layer="91"/>
 </segment>
 </net>
@@
 <wire x1="71.12" y1="144.78" x2="71.12" y2="137.62" width="0.1524" layer="91"/>
 </segment>
+<segment>
+<pinref part="P+3" gate="1" pin="+5V"/>
+<wire x1="116.84" y1="144.78" x2="116.84" y2="139.7" width="0.1524" layer="91"/>
+<pinref part="J1" gate="G$1" pin="1"/>
+<wire x1="116.84" y1="139.7" x2="119.38" y2="139.7" width="0.1524" layer="91"/>
+</segment>
 </net>
